Commit message: CartesioTestsCpp-added new coman urdf srdf file

File: CartesioTestsCpp/robots/coman/urdf/coman.urdf (robot description, URDF)
Before this commit: robot coman, 65 links, 64 joints
Links:
- link DWL: geometry collision mesh filename=package://coman_urdf/meshes/simple/Torso1.STL scale=0.03937 0.03937 0.03937; visual mesh filename=package://coman_urdf/meshes/Torso1.STL scale=0.03937 0.03937 0.03937
- link DWS: geometry collision mesh filename=package://coman_urdf/meshes/simple/Torso2.STL scale=0.03937 0.03937 0.03937; visual mesh filename=package://coman_urdf/meshes/Torso2.STL scale=0.03937 0.03937 0.03937
- link DWYTorso: geometry collision mesh filename=package://coman_urdf/meshes/simple/Torso3.STL scale=0.03937 0.03937 0.03937; visual mesh filename=package://coman_urdf/meshes/Torso3.STL scale=0.03937 0.03937 0.03937
- link LElb: geometry collision mesh filename=package://coman_urdf/meshes/simple/Elbow.STL scale=1.0 1.0 1.0; visual mesh filename=package://coman_urdf/meshes/Elbow.STL scale=1.0 1.0 1.0
- link LFootmot: geometry collision mesh filename=package://coman_urdf/meshes/simple/Leg4.STL scale=0.03937 -0.03937 0.03937; visual mesh filename=package://coman_urdf/meshes/Leg4.STL scale=0.03937 -0.03937 0.03937
- link LForearm: geometry collision mesh filename=package://coman_urdf/meshes/simple/Forearm0.STL scale=1.0 1.0 1.0; visual mesh filename=package://coman_urdf/meshes/Forearm0.STL scale=0.1 0.1 0.1
- link LHipMot: geometry collision mesh filename=package://coman_urdf/meshes/simple/Leg0.STL scale=0.03937 -0.03937 0.03937; visual mesh filename=package://coman_urdf/meshes/Leg0.STL scale=0.03937 -0.03937 0.03937
- link LLowLeg: geometry collision mesh filename=package://coman_urdf/meshes/simple/Leg3.STL scale=0.03937 -0.03937 0.03937; visual mesh filename=package://coman_urdf/meshes/Leg3.STL scale=0.03937 -0.03937 0.03937
- link LShp: geometry collision mesh filename=package://coman_urdf/meshes/simple/Arm0.STL scale=0.03937 -0.03937 0.03937; visual mesh filename=package://coman_urdf/meshes/Arm0.STL scale=0.03937 -0.03937 0.03937
- link LShr: geometry collision mesh filename=package://coman_urdf/meshes/simple/Arm1.STL scale=0.03937 -0.03937 0.03937; visual mesh filename=package://coman_urdf/meshes/Arm1.STL scale=0.03937 -0.03937 0.03937
- link LShy: geometry collision mesh filename=package://coman_urdf/meshes/simple/Arm2.STL scale=0.03937 -0.03937 0.03937; visual mesh filename=package://coman_urdf/meshes/Arm2.STL scale=0.03937 -0.03937 0.03937
- link LSoftHand: geometry collision mesh filename=package://coman_urdf/meshes/simple/SoftHandOpen.STL scale=-1E-3 1E-3 1E-3; visual mesh filename=package://coman_urdf/meshes/SoftHandOpen.STL scale=-0.1 0.1 0.1
- link LThighLowLeg: geometry collision mesh filename=package://coman_urdf/meshes/simple/Leg2.STL scale=0.03937 -0.03937 0.03937; visual mesh filename=package://coman_urdf/meshes/Leg2.STL scale=0.03937 -0.03937 0.03937
- link LThighUpLeg: geometry collision mesh filename=package://coman_urdf/meshes/simple/Leg1.STL scale=0.03937 -0.03937 0.03937; visual mesh filename=package://coman_urdf/meshes/Leg1.STL scale=0.03937 -0.03937 0.03937
- link LWrMot2: geometry collision mesh filename=package://coman_urdf/meshes/simple/Forearm1.STL scale=0.001 0.001 0.001; visual mesh filename=package://coman_urdf/meshes/Forearm1.STL scale=0.001 0.001 0.001
- link LWrMot3: geometry collision mesh filename=package://coman_urdf/meshes/simple/Forearm2.STL scale=0.001 0.001 0.001; visual mesh filename=package://coman_urdf/meshes/Forearm2.STL scale=0.001 0.001 0.001
- link RElb: geometry collision mesh filename=package://coman_urdf/meshes/simple/Elbow.STL scale=1.0 1.0 1.0; visual mesh filename=package://coman_urdf/meshes/Elbow.STL scale=1.0 1.0 1.0
- link RFootmot: geometry collision mesh filename=package://coman_urdf/meshes/simple/Leg4.STL scale=0.03937 0.03937 0.03937; visual mesh filename=package://coman_urdf/meshes/Leg4.STL scale=0.03937 0.03937 0.03937
- link RForearm: geometry collision mesh filename=package://coman_urdf/meshes/simple/Forearm0.STL scale=1.0 1.0 1.0; visual mesh filename=package://coman_urdf/meshes/Forearm0.STL scale=0.1 0.1 0.1
- link RHipMot: geometry collision mesh filename=package://coman_urdf/meshes/simple/Leg0.STL scale=0.03937 0.03937 0.03937; visual mesh filename=package://coman_urdf/meshes/Leg0.STL scale=0.03937 0.03937 0.03937
- link RLowLeg: geometry collision mesh filename=package://coman_urdf/meshes/simple/Leg3.STL scale=0.03937 0.03937 0.03937; visual mesh filename=package://coman_urdf/meshes/Leg3.STL scale=0.03937 0.03937 0.03937
- link RShp: geometry collision mesh filename=package://coman_urdf/meshes/simple/Arm0.STL scale=0.03937 0.03937 0.03937; visual mesh filename=package://coman_urdf/meshes/Arm0.STL scale=0.03937 0.03937 0.03937
- link RShr: geometry collision mesh filename=package://coman_urdf/meshes/simple/Arm1.STL scale=0.03937 0.03937 0.03937; visual mesh filename=package://coman_urdf/meshes/Arm1.STL scale=0.03937 0.03937 0.03937
- link RShy: geometry collision mesh filename=package://coman_urdf/meshes/simple/Arm2.STL scale=0.03937 0.03937 0.03937; visual mesh filename=package://coman_urdf/meshes/Arm2.STL scale=0.03937 0.03937 0.03937
- link RSoftHand: geometry collision mesh filename=package://coman_urdf/meshes/simple/SoftHandOpen.STL scale=1E-3 1E-3 1E-3; visual mesh filename=package://coman_urdf/meshes/SoftHandOpen.STL scale=0.1 0.1 0.1
- link RThighLowLeg: geometry collision mesh filename=package://coman_urdf/meshes/simple/Leg2.STL scale=0.03937 0.03937 0.03937; visual mesh filename=package://coman_urdf/meshes/Leg2.STL scale=0.03937 0.03937 0.03937
- link RThighUpLeg: geometry collision mesh filename=package://coman_urdf/meshes/simple/Leg1.STL scale=0.03937 0.03937 0.03937; visual mesh filename=package://coman_urdf/meshes/Leg1.STL scale=0.03937 0.03937 0.03937
- link RWrMot2: geometry collision mesh filename=package://coman_urdf/meshes/simple/Forearm1.STL scale=0.001 0.001 0.001; visual mesh filename=package://coman_urdf/meshes/Forearm1.STL scale=0.001 0.001 0.001
- link RWrMot3: geometry collision mesh filename=package://coman_urdf/meshes/simple/Forearm2.STL scale=0.001 0.001 0.001; visual mesh filename=package://coman_urdf/meshes/Forearm2.STL scale=0.001 0.001 0.001
- link Waist: geometry collision mesh filename=package://coman_urdf/meshes/simple/Waist.STL scale=0.03937 0.03937 0.03937; visual mesh filename=package://coman_urdf/meshes/Waist.STL scale=0.03937 0.03937 0.03937
Joints:
- joint imu_joint: origin xyz=-0.072 -0.0068 0.044 rpy=0 0 0 -> xyz=-0.072 -0.0068 0.044 rpy=1.57079632679 0 1.57079632679
