Commit message: CartesioTestsCpp- fixed rviz visualization meshes error

File: CartesioTestsCpp/robots/centauro/urdf/centauro.urdf (robot description, URDF)
Before this commit: robot centauro, 54 links, 53 joints
Links:
- link ankle1_1: geometry collision mesh filename=file:///home/liana/catkin_ws/src/CartesioTests/CartesioTest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 scale=0.001 0.001 0.001; visual mesh filename=file:///home/liana/catkin_ws/src/CartesioTests/CartesioTest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 scale=0.001 0.001 0.001
- link ankle1_2: geometry collision mesh filename=file:///home/liana/catkin_ws/src/CartesioTests/CartesioTest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 scale=0.001 0.001 0.001; visual mesh filename=file:///home/liana/catkin_ws/src/CartesioTests/CartesioTest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 scale=0.001 0.001 0.001
- link ankle1_3: geometry collision mesh filename=file:///home/liana/catkin_ws/src/CartesioTests/CartesioTest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 scale=0.001 0.001 0.001; visual mesh filename=file:///home/liana/catkin_ws/src/CartesioTests/CartesioTest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 scale=0.001 0.001 0.001
- link ankle1_4: geometry collision mesh filename=file:///home/liana/catkin_ws/src/CartesioTests/CartesioTest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 scale=0.001 0.001 0.001; visual mesh filename=file:///home/liana/catkin_ws/src/CartesioTests/CartesioTest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 scale=0.001 0.001 0.001
- link ankle2_1: geometry collision mesh filename=file:///home/liana/catkin_ws/src/CartesioTests/CartesioTest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 scale=0.001 0.001 0.001; visual mesh filename=file:///home/liana/catkin_ws/src/CartesioTests/CartesioTest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 scale=0.001 0.001 0.001
- link ankle2_2: geometry collision mesh filename=file:///home/liana/catkin_ws/src/CartesioTests/CartesioTest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 scale=0.001 0.001 0.001; visual mesh filename=file:///home/liana/catkin_ws/src/CartesioTests/CartesioTest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 scale=0.001 0.001 0.001
- link ankle2_3: geometry collision mesh filename=file:///home/liana/catkin_ws/src/CartesioTests/CartesioTest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 scale=0.001 0.001 0.001; visual mesh filename=file:///home/liana/catkin_ws/src/CartesioTests/CartesioTest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 scale=0.001 0.001 0.001
- link ankle2_4: geometry collision mesh filename=file:///home/liana/catkin_ws/src/CartesioTests/CartesioTest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 scale=0.001 0.001 0.001; visual mesh filename=file:///home/liana/catkin_ws/src/CartesioTests/CartesioTest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 scale=0.001 0.001 0.001
- link arm1_1: geometry collision mesh filename=file:///home/liana/catkin_ws/src/CartesioTests/CartesioTest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 scale=0.001 -0.001 0.001; visual mesh filename=file:///home/liana/catkin_ws/src/CartesioTests/CartesioTest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 scale=0.001 -0.001 0.001
- link arm1_2: geometry collision mesh filename=file:///home/liana/catkin_ws/src/CartesioTests/CartesioTest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 scale=0.001 -0.001 0.001; visual mesh filename=file:///home/liana/catkin_ws/src/CartesioTests/CartesioTest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 scale=0.001 -0.001 0.001
- link arm1_3: geometry collision mesh filename=file:///home/liana/catkin_ws/src/CartesioTests/CartesioTest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 scale=0.001 -0.001 0.001; visual mesh filename=file:///home/liana/catkin_ws/src/CartesioTests/CartesioTest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 scale=0.001 -0.001 0.001
- link arm1_4: geometry collision mesh filename=file:///home/liana/catkin_ws/src/CartesioTests/CartesioTest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 scale=0.001 -0.001 0.001; visual mesh filename=file:///home/liana/catkin_ws/src/CartesioTests/CartesioTest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 scale=0.001 -0.001 0.001
- link arm1_5: geometry collision mesh filename=file:///home/liana/catkin_ws/src/CartesioTests/CartesioTest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 scale=0.001 -0.001 0.001; visual mesh filename=file:///home/liana/catkin_ws/src/CartesioTests/CartesioTest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 scale=0.001 -0.001 0.001
- link arm1_6: geometry collision mesh filename=file:///home/liana/catkin_ws/src/CartesioTests/CartesioTest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 scale=0.001 -0.001 0.001; visual mesh filename=file:///home/liana/catkin_ws/src/CartesioTests/CartesioTest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 scale=0.001 -0.001 0.001
- link arm1_7: geometry collision mesh filename=file:///home/liana/catkin_ws/src/CartesioTests/CartesioTest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 scale=0.001 -0.001 0.001; visual mesh filename=file:///home/liana/catkin_ws/src/CartesioTests/CartesioTest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 scale=0.001 -0.001 0.001
- link arm2_1: geometry collision mesh filename=file:///home/liana/catkin_ws/src/CartesioTests/CartesioTest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 scale=0.001 0.001 0.001; visual mesh filename=file:///home/liana/catkin_ws/src/CartesioTests/CartesioTest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 scale=0.001 0.001 0.001
- link arm2_2: geometry collision mesh filename=file:///home/liana/catkin_ws/src/CartesioTests/CartesioTest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 scale=0.001 0.001 0.001; visual mesh filename=file:///home/liana/catkin_ws/src/CartesioTests/CartesioTest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 scale=0.001 0.001 0.001
- link arm2_3: geometry collision mesh filename=file:///home/liana/catkin_ws/src/CartesioTests/CartesioTest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 scale=0.001 0.001 0.001; visual mesh filename=file:///home/liana/catkin_ws/src/CartesioTests/CartesioTest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 scale=0.001 0.001 0.001
- link arm2_4: geometry collision mesh filename=file:///home/liana/catkin_ws/src/CartesioTests/CartesioTest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 scale=0.001 0.001 0.001; visual mesh filename=file:///home/liana/catkin_ws/src/CartesioTests/CartesioTest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 scale=0.001 0.001 0.001
- link arm2_5: geometry collision mesh filename=file:///home/liana/catkin_ws/src/CartesioTests/CartesioTest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 scale=0.001 0.001 0.001; visual mesh filename=file:///home/liana/catkin_ws/src/CartesioTests/CartesioTest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 scale=0.001 0.001 0.001
- link arm2_6: geometry collision mesh filename=file:///home/liana/catkin_ws/src/CartesioTests/CartesioTest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 scale=0.001 0.001 0.001; visual mesh filename=file:///home/liana/catkin_ws/src/CartesioTests/CartesioTest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 scale=0.001 0.001 0.001
- link arm2_7: geometry collision mesh filename=file:///home/liana/catkin_ws/src/CartesioTests/CartesioTest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 scale=0.001 0.001 0.001; visual mesh filename=file:///home/liana/catkin_ws/src/CartesioTests/CartesioTest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 scale=0.001 0.001 0.001
- link ball1: geometry collision mesh filename=file:///home/liana/catkin_ws/src/CartesioTests/CartesioTest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 scale=0.001 0.001 0.001; visual mesh filename=file:///home/liana/catkin_ws/src/CartesioTests/CartesioTest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 scale=0.001 0.001 0.001
- link ball2: geometry collision mesh filename=file:///home/liana/catkin_ws/src/CartesioTests/CartesioTest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 scale=0.001 0.001 0.001; visual mesh filename=file:///home/liana/catkin_ws/src/CartesioTests/CartesioTest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 scale=0.001 0.001 0.001
- link hip1_1: geometry collision mesh filename=file:///home/liana/catkin_ws/src/CartesioTests/CartesioTest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 scale=0.001 0.001 0.001; visual mesh filename=file:///home/liana/catkin_ws/src/CartesioTests/CartesioTest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 scale=0.001 0.001 0.001
- link hip1_2: geometry collision mesh filename=file:///home/liana/catkin_ws/src/CartesioTests/CartesioTest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 scale=0.001 0.001 0.001; visual mesh filename=file:///home/liana/catkin_ws/src/CartesioTests/CartesioTest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 scale=0.001 0.001 0.001
- link hip1_3: geometry collision mesh filename=file:///home/liana/catkin_ws/src/CartesioTests/CartesioTest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 scale=0.001 0.001 0.001; visual mesh filename=file:///home/liana/catkin_ws/src/CartesioTests/CartesioTest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 scale=0.001 0.001 0.001
- link hip1_4: geometry collision mesh filename=file:///home/liana/catkin_ws/src/CartesioTests/CartesioTest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 scale=0.001 0.001 0.001; visual mesh filename=file:///home/liana/catkin_ws/src/CartesioTests/CartesioTest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 scale=0.001 0.001 0.001
- link hip2_1: geometry collision mesh filename=file:///home/liana/catkin_ws/src/CartesioTests/CartesioTest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 scale=0.001 0.001 0.001; visual mesh filename=file:///home/liana/catkin_ws/src/CartesioTests/CartesioTest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 scale=0.001 0.001 0.001
- link hip2_2: geometry collision mesh filename=file:///home/liana/catkin_ws/src/CartesioTests/CartesioTest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 scale=0.001 0.001 0.001; visual mesh filename=file:///home/liana/catkin_ws/src/CartesioTests/CartesioTest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 scale=0.001 0.001 0.001
- link hip2_3: geometry collision mesh filename=file:///home/liana/catkin_ws/src/CartesioTests/CartesioTest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 scale=0.001 0.001 0.001; visual mesh filename=file:///home/liana/catkin_ws/src/CartesioTests/CartesioTest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 scale=0.001 0.001 0.001
- link hip2_4: geometry collision mesh filename=file:///home/liana/catkin_ws/src/CartesioTests/CartesioTest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 scale=0.001 0.001 0.001; visual mesh filename=file:///home/liana/catkin_ws/src/CartesioTests/CartesioTest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 scale=0.001 0.001 0.001
- link knee_1: geometry collision mesh filename=file:///home/liana/catkin_ws/src/CartesioTests/CartesioTest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 scale=0.001 0.001 0.001; visual mesh filename=file:///home/liana/catkin_ws/src/CartesioTests/CartesioTest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 scale=0.001 0.001 0.001
- link knee_2: geometry collision mesh filename=file:///home/liana/catkin_ws/src/CartesioTests/CartesioTest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 scale=0.001 0.001 0.001; visual mesh filename=file:///home/liana/catkin_ws/src/CartesioTests/CartesioTest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 scale=0.001 0.001 0.001
- link knee_3: geometry collision mesh filename=file:///home/liana/catkin_ws/src/CartesioTests/CartesioTest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 scale=0.001 0.001 0.001; visual mesh filename=file:///home/liana/catkin_ws/src/CartesioTests/CartesioTest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 scale=0.001 0.001 0.001
- link knee_4: geometry collision mesh filename=file:///home/liana/catkin_ws/src/CartesioTests/CartesioTest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 scale=0.001 0.001 0.001; visual mesh filename=file:///home/liana/catkin_ws/src/CartesioTests/CartesioTest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 scale=0.001 0.001 0.001
- link neck_1: geometry collision mesh filename=file:///home/liana/catkin_ws/src/CartesioTests/CartesioTest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 scale=0.001 0.001 0.001; visual mesh filename=file:///home/liana/catkin_ws/src/CartesioTests/CartesioTest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 scale=0.001 0.001 0.001
- link neck_2: geometry collision mesh filename=file:///home/liana/catkin_ws/src/CartesioTests/CartesioTest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 scale=0.001 0.001 0.001; visual mesh filename=file:///home/liana/catkin_ws/src/CartesioTests/CartesioTest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 scale=0.001 0.001 0.001
- link neck_3: geometry collision mesh filename=file:///home/liana/catkin_ws/src/CartesioTests/CartesioTest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 scale=0.001 0.001 0.001; visual mesh filename=file:///home/liana/catkin_ws/src/CartesioTests/CartesioTest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 scale=0.001 0.001 0.001
- link pelvis: geometry collision mesh filename=file:///home/liana/catkin_ws/src/CartesioTests/CartesioTest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 scale=0.001 0.001 0.001; visual mesh filename=file:///home/liana/catkin_ws/src/CartesioTests/CartesioTest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 scale=0.001 0.001 0.001
- link torso_2: geometry collision mesh filename=file:///home/liana/catkin_ws/src/CartesioTests/CartesioTest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 scale=0.001 0.001 0.001; visual mesh filename=file:///home/liana/catkin_ws/src/CartesioTests/CartesioTest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 scale=0.001 0.001 0.001
- link wheel_1: geometry collision cylinder length=0.06 radius=0.078; visual mesh filename=file:///home/liana/catkin_ws/src/CartesioTests/CartesioTest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 scale=0.001 0.001 0.001
- link wheel_2: geometry collision cylinder length=0.06 radius=0.078; visual mesh filename=file:///home/liana/catkin_ws/src/CartesioTests/CartesioTest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 scale=0.001 0.001 0.001
- link wheel_3: geometry collision cylinder length=0.06 radius=0.078; visual mesh filename=file:///home/liana/catkin_ws/src/CartesioTests/CartesioTest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 scale=0.001 0.001 0.001
- link wheel_4: geometry collision cylinder length=0.06 radius=0.078; visual mesh filename=file:///home/liana/catkin_ws/src/CartesioTests/CartesioTest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 scale=0.001 0.001 0.001

File: CartesioTestsCpp/robots/coman/urdf/coman.urdf (robot description, URDF)
Before this commit: robot coman, 65 links, 64 joints
Links:
- link DWL: geometry collision mesh filename=file:///home/liana/catkin_ws/src/CartesioTests/CartesioTest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 scale=0.03937 0.03937 0.03937; visual mesh filename=file:///home/liana/catkin_ws/src/CartesioTests/CartesioTest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 scale=0.03937 0.03937 0.03937
- link DWS: geometry collision mesh filename=file:///home/liana/catkin_ws/src/CartesioTests/CartesioTest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 scale=0.03937 0.03937 0.03937; visual mesh filename=file:///home/liana/catkin_ws/src/CartesioTests/CartesioTest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 scale=0.03937 0.03937 0.03937
- link DWYTorso: geometry collision mesh filename=file:///home/liana/catkin_ws/src/CartesioTests/CartesioTest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 scale=0.03937 0.03937 0.03937; visual mesh filename=file:///home/liana/catkin_ws/src/CartesioTests/CartesioTest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 scale=0.03937 0.03937 0.03937
- link LElb: geometry collision mesh filename=file:///home/liana/catkin_ws/src/CartesioTests/CartesioTest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 scale=1.0 1.0 1.0; visual mesh filename=file:///home/liana/catkin_ws/src/CartesioTests/CartesioTest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 scale=1.0 1.0 1.0
- link LFootmot: geometry collision mesh filename=file:///home/liana/catkin_ws/src/CartesioTests/CartesioTest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 scale=0.03937 -0.03937 0.03937; visual mesh filename=file:///home/liana/catkin_ws/src/CartesioTests/CartesioTest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 scale=0.03937 -0.03937 0.03937
- link LForearm: geometry collision mesh filename=file:///home/liana/catkin_ws/src/CartesioTests/CartesioTest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 scale=1.0 1.0 1.0; visual mesh filename=file:///home/liana/catkin_ws/src/CartesioTests/CartesioTest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 scale=0.1 0.1 0.1
- link LHipMot: geometry collision mesh filename=file:///home/liana/catkin_ws/src/CartesioTests/CartesioTest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 scale=0.03937 -0.03937 0.03937; visual mesh filename=file:///home/liana/catkin_ws/src/CartesioTests/CartesioTest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 scale=0.03937 -0.03937 0.03937
- link LLowLeg: geometry collision mesh filename=file:///home/liana/catkin_ws/src/CartesioTests/CartesioTest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 scale=0.03937 -0.03937 0.03937; visual mesh filename=file:///home/liana/catkin_ws/src/CartesioTests/CartesioTest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 scale=0.03937 -0.03937 0.03937
- link LShp: geometry collision mesh filename=file:///home/liana/catkin_ws/src/CartesioTests/CartesioTest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 scale=0.03937 -0.03937 0.03937; visual mesh filename=file:///home/liana/catkin_ws/src/CartesioTests/CartesioTest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 scale=0.03937 -0.03937 0.03937
- link LShr: geometry collision mesh filename=file:///home/liana/catkin_ws/src/CartesioTests/CartesioTest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 scale=0.03937 -0.03937 0.03937; visual mesh filename=file:///home/liana/catkin_ws/src/CartesioTests/CartesioTest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 scale=0.03937 -0.03937 0.03937
- link LShy: geometry collision mesh filename=file:///home/liana/catkin_ws/src/CartesioTests/CartesioTest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 scale=0.03937 -0.03937 0.03937; visual mesh filename=file:///home/liana/catkin_ws/src/CartesioTests/CartesioTest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 scale=0.03937 -0.03937 0.03937
- link LSoftHand: geometry collision mesh filename=file:///home/liana/catkin_ws/src/CartesioTests/CartesioTest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 scale=-1E-3 1E-3 1E-3; visual mesh filename=file:///home/liana/catkin_ws/src/CartesioTests/CartesioTest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 scale=-0.1 0.1 0.1
- link LThighLowLeg: geometry collision mesh filename=file:///home/liana/catkin_ws/src/CartesioTests/CartesioTest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 scale=0.03937 -0.03937 0.03937; visual mesh filename=file:///home/liana/catkin_ws/src/CartesioTests/CartesioTest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 scale=0.03937 -0.03937 0.03937
- link LThighUpLeg: geometry collision mesh filename=file:///home/liana/catkin_ws/src/CartesioTests/CartesioTest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 scale=0.03937 -0.03937 0.03937; visual mesh filename=file:///home/liana/catkin_ws/src/CartesioTests/CartesioTest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 scale=0.03937 -0.03937 0.03937
- link LWrMot2: geometry collision mesh filename=file:///home/liana/catkin_ws/src/CartesioTests/CartesioTest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 scale=0.001 0.001 0.001; visual mesh filename=file:///home/liana/catkin_ws/src/CartesioTests/CartesioTest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 scale=0.001 0.001 0.001
- link LWrMot3: geometry collision mesh filename=file:///home/liana/catkin_ws/src/CartesioTests/CartesioTest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 scale=0.001 0.001 0.001; visual mesh filename=file:///home/liana/catkin_ws/src/CartesioTests/CartesioTest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 scale=0.001 0.001 0.001
- link RElb: geometry collision mesh filename=file:///home/liana/catkin_ws/src/CartesioTests/CartesioTest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 scale=1.0 1.0 1.0; visual mesh filename=file:///home/liana/catkin_ws/src/CartesioTests/CartesioTest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 scale=1.0 1.0 1.0
- link RFootmot: geometry collision mesh filename=file:///home/liana/catkin_ws/src/CartesioTests/CartesioTest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 scale=0.03937 0.03937 0.03937; visual mesh filename=file:///home/liana/catkin_ws/src/CartesioTests/CartesioTest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 scale=0.03937 0.03937 0.03937
- link RForearm: geometry collision mesh filename=file:///home/liana/catkin_ws/src/CartesioTests/CartesioTest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 scale=1.0 1.0 1.0; visual mesh filename=file:///home/liana/catkin_ws/src/CartesioTests/CartesioTest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 scale=0.1 0.1 0.1
- link RHipMot: geometry collision mesh filename=file:///home/liana/catkin_ws/src/CartesioTests/CartesioTest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 scale=0.03937 0.03937 0.03937; visual mesh filename=file:///home/liana/catkin_ws/src/CartesioTests/CartesioTest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 scale=0.03937 0.03937 0.03937
- link RLowLeg: geometry collision mesh filename=file:///home/liana/catkin_ws/src/CartesioTests/CartesioTest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 scale=0.03937 0.03937 0.03937; visual mesh filename=file:///home/liana/catkin_ws/src/CartesioTests/CartesioTest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 scale=0.03937 0.03937 0.03937
- link RShp: geometry collision mesh filename=file:///home/liana/catkin_ws/src/CartesioTests/CartesioTest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 scale=0.03937 0.03937 0.03937; visual mesh filename=file:///home/liana/catkin_ws/src/CartesioTests/CartesioTest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 scale=0.03937 0.03937 0.03937
- link RShr: geometry collision mesh filename=file:///home/liana/catkin_ws/src/CartesioTests/CartesioTest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 scale=0.03937 0.03937 0.03937; visual mesh filename=file:///home/liana/catkin_ws/src/CartesioTests/CartesioTest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 scale=0.03937 0.03937 0.03937
- link RShy: geometry collision mesh filename=file:///home/liana/catkin_ws/src/CartesioTests/CartesioTest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 scale=0.03937 0.03937 0.03937; visual mesh filename=file:///home/liana/catkin_ws/src/CartesioTests/CartesioTest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 scale=0.03937 0.03937 0.03937
- link RSoftHand: geometry collision mesh filename=file:///home/liana/catkin_ws/src/CartesioTests/CartesioTest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 scale=1E-3 1E-3 1E-3; visual mesh filename=file:///home/liana/catkin_ws/src/CartesioTests/CartesioTest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 scale=0.1 0.1 0.1
- link RThighLowLeg: geometry collision mesh filename=file:///home/liana/catkin_ws/src/CartesioTests/CartesioTest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 scale=0.03937 0.03937 0.03937; visual mesh filename=file:///home/liana/catkin_ws/src/CartesioTests/CartesioTest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 scale=0.03937 0.03937 0.03937
- link RThighUpLeg: geometry collision mesh filename=file:///home/liana/catkin_ws/src/CartesioTests/CartesioTest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 scale=0.03937 0.03937 0.03937; visual mesh filename=file:///home/liana/catkin_ws/src/CartesioTests/CartesioTest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 scale=0.03937 0.03937 0.03937
- link RWrMot2: geometry collision mesh filename=file:///home/liana/catkin_ws/src/CartesioTests/CartesioTest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 scale=0.001 0.001 0.001; visual mesh filename=file:///home/liana/catkin_ws/src/CartesioTests/CartesioTest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 scale=0.001 0.001 0.001
- link RWrMot3: geometry collision mesh filename=file:///home/liana/catkin_ws/src/CartesioTests/CartesioTest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 scale=0.001 0.001 0.001; visual mesh filename=file:///home/liana/catkin_ws/src/CartesioTests/CartesioTest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 scale=0.001 0.001 0.001
- link Waist: geometry collision mesh filename=file:///home/liana/catkin_ws/src/CartesioTests/CartesioTest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 scale=0.03937 0.03937 0.03937; visual mesh filename=file:///home/liana/catkin_ws/src/CartesioTests/CartesioTest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 scale=0.03937 0.03937 0.03937
