Commit message: added launch file for centauro in cartesio tests quick start

File: CartesioTestsQuickStart/robots/centauro/urdf/centauro.urdf (robot description, URDF)
Before this commit: robot centauro, 54 links, 53 joints
Links:
- link ankle1_1: geometry collision mesh filename=package://vir_singlejoint/robots/centauro/meshes/simple/ank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 scale=0.001 0.001 0.001; visual mesh filename=package://vir_singlejoint/robots/centauro/meshes/ankle-pitc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 scale=0.001 0.001 0.001
- link ankle1_2: geometry collision mesh filename=package://vir_singlejoint/robots/centauro/meshes/simple/ank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 scale=0.001 0.001 0.001; visual mesh filename=package://vir_singlejoint/robots/centauro/meshes/ankle-pitc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 scale=0.001 0.001 0.001
- link ankle1_3: geometry collision mesh filename=package://vir_singlejoint/robots/centauro/meshes/simple/ank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 scale=0.001 0.001 0.001; visual mesh filename=package://vir_singlejoint/robots/centauro/meshes/ankle-pitc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 scale=0.001 0.001 0.001
- link ankle1_4: geometry collision mesh filename=package://vir_singlejoint/robots/centauro/meshes/simple/ank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 scale=0.001 0.001 0.001; visual mesh filename=package://vir_singlejoint/robots/centauro/meshes/ankle-pitc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 scale=0.001 0.001 0.001
- link ankle2_1: geometry collision mesh filename=package://vir_singlejoint/robots/centauro/meshes/simple/ank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 scale=0.001 0.001 0.001; visual mesh filename=package://vir_singlejoint/robots/centauro/meshes/ankle-yaw.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 scale=0.001 0.001 0.001
- link ankle2_2: geometry collision mesh filename=package://vir_singlejoint/robots/centauro/meshes/simple/ank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 scale=0.001 0.001 0.001; visual mesh filename=package://vir_singlejoint/robots/centauro/meshes/ankle-yaw.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 scale=0.001 0.001 0.001
- link ankle2_3: geometry collision mesh filename=package://vir_singlejoint/robots/centauro/meshes/simple/ank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 scale=0.001 0.001 0.001; visual mesh filename=package://vir_singlejoint/robots/centauro/meshes/ankle-yaw.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 scale=0.001 0.001 0.001
- link ankle2_4: geometry collision mesh filename=package://vir_singlejoint/robots/centauro/meshes/simple/ank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 scale=0.001 0.001 0.001; visual mesh filename=package://vir_singlejoint/robots/centauro/meshes/ankle-yaw.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 scale=0.001 0.001 0.001
- link arm1_1: geometry collision mesh filename=package://vir_singlejoint/robots/centauro/meshes/simple/Sho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 scale=0.001 -0.001 0.001; visual mesh filename=package://vir_singlejoint/robots/centauro/meshes/ShoulderPi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 scale=0.001 -0.001 0.001
- link arm1_2: geometry collision mesh filename=package://vir_singlejoint/robots/centauro/meshes/simple/Sho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 scale=0.001 -0.001 0.001; visual mesh filename=package://vir_singlejoint/robots/centauro/meshes/ShoulderRo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 scale=0.001 -0.001 0.001
- link arm1_3: geometry collision mesh filename=package://vir_singlejoint/robots/centauro/meshes/simple/Sho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 scale=0.001 -0.001 0.001; visual mesh filename=package://vir_singlejoint/robots/centauro/meshes/ShoulderYa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 scale=0.001 -0.001 0.001
- link arm1_4: geometry collision mesh filename=package://vir_singlejoint/robots/centauro/meshes/simple/Elb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 scale=0.001 -0.001 0.001; visual mesh filename=package://vir_singlejoint/robots/centauro/meshes/Elbow.STL scale=0.001 -0.001 0.001
- link arm1_5: geometry collision mesh filename=package://vir_singlejoint/robots/centauro/meshes/simple/For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 scale=0.001 -0.001 0.001; visual mesh filename=package://vir_singlejoint/robots/centauro/meshes/Forearm.STL scale=0.001 -0.001 0.001
- link arm1_6: geometry collision mesh filename=package://vir_singlejoint/robots/centauro/meshes/simple/For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 scale=0.001 -0.001 0.001; visual mesh filename=package://vir_singlejoint/robots/centauro/meshes/ForearmPit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 scale=0.001 -0.001 0.001
- link arm1_7: geometry collision mesh filename=package://vir_singlejoint/robots/centauro/meshes/simple/For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 scale=0.001 -0.001 0.001; visual mesh filename=package://vir_singlejoint/robots/centauro/meshes/ForearmYaw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 scale=0.001 -0.001 0.001
- link arm2_1: geometry collision mesh filename=package://vir_singlejoint/robots/centauro/meshes/simple/Sho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 scale=0.001 0.001 0.001; visual mesh filename=package://vir_singlejoint/robots/centauro/meshes/ShoulderPi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 scale=0.001 0.001 0.001
- link arm2_2: geometry collision mesh filename=package://vir_singlejoint/robots/centauro/meshes/simple/Sho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 scale=0.001 0.001 0.001; visual mesh filename=package://vir_singlejoint/robots/centauro/meshes/ShoulderRo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 scale=0.001 0.001 0.001
- link arm2_3: geometry collision mesh filename=package://vir_singlejoint/robots/centauro/meshes/simple/Sho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 scale=0.001 0.001 0.001; visual mesh filename=package://vir_singlejoint/robots/centauro/meshes/ShoulderYa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 scale=0.001 0.001 0.001
- link arm2_4: geometry collision mesh filename=package://vir_singlejoint/robots/centauro/meshes/simple/Elb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 scale=0.001 0.001 0.001; visual mesh filename=package://vir_singlejoint/robots/centauro/meshes/Elbow.STL scale=0.001 0.001 0.001
- link arm2_5: geometry collision mesh filename=package://vir_singlejoint/robots/centauro/meshes/simple/For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 scale=0.001 0.001 0.001; visual mesh filename=package://vir_singlejoint/robots/centauro/meshes/Forearm.STL scale=0.001 0.001 0.001
- link arm2_6: geometry collision mesh filename=package://vir_singlejoint/robots/centauro/meshes/simple/For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 scale=0.001 0.001 0.001; visual mesh filename=package://vir_singlejoint/robots/centauro/meshes/ForearmPit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 scale=0.001 0.001 0.001
- link arm2_7: geometry collision mesh filename=package://vir_singlejoint/robots/centauro/meshes/simple/For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 scale=0.001 0.001 0.001; visual mesh filename=package://vir_singlejoint/robots/centauro/meshes/ForearmYaw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 scale=0.001 0.001 0.001
- link ball1: geometry collision mesh filename=package://vir_singlejoint/robots/centauro/meshes/simple/Bal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 scale=0.001 0.001 0.001; visual mesh filename=package://vir_singlejoint/robots/centauro/meshes/BallHand.s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 scale=0.001 0.001 0.001
- link ball2: geometry collision mesh filename=package://vir_singlejoint/robots/centauro/meshes/simple/Bal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 scale=0.001 0.001 0.001; visual mesh filename=package://vir_singlejoint/robots/centauro/meshes/BallHand.s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 scale=0.001 0.001 0.001
- link hip1_1: geometry collision mesh filename=package://vir_singlejoint/robots/centauro/meshes/simple/hip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 scale=0.001 0.001 0.001; visual mesh filename=package://vir_singlejoint/robots/centauro/meshes/hip-yaw.stl scale=0.001 0.001 0.001
- link hip1_2: geometry collision mesh filename=package://vir_singlejoint/robots/centauro/meshes/simple/hip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 scale=0.001 0.001 0.001; visual mesh filename=package://vir_singlejoint/robots/centauro/meshes/hip-yaw.stl scale=0.001 0.001 0.001
- link hip1_3: geometry collision mesh filename=package://vir_singlejoint/robots/centauro/meshes/simple/hip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 scale=0.001 0.001 0.001; visual mesh filename=package://vir_singlejoint/robots/centauro/meshes/hip-yaw.stl scale=0.001 0.001 0.001
- link hip1_4: geometry collision mesh filename=package://vir_singlejoint/robots/centauro/meshes/simple/hip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 scale=0.001 0.001 0.001; visual mesh filename=package://vir_singlejoint/robots/centauro/meshes/hip-yaw.stl scale=0.001 0.001 0.001
- link hip2_1: geometry collision mesh filename=package://vir_singlejoint/robots/centauro/meshes/simple/hip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 scale=0.001 0.001 0.001; visual mesh filename=package://vir_singlejoint/robots/centauro/meshes/hip-pitch.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 scale=0.001 0.001 0.001
- link hip2_2: geometry collision mesh filename=package://vir_singlejoint/robots/centauro/meshes/simple/hip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 scale=0.001 0.001 0.001; visual mesh filename=package://vir_singlejoint/robots/centauro/meshes/hip-pitch.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 scale=0.001 0.001 0.001
- link hip2_3: geometry collision mesh filename=package://vir_singlejoint/robots/centauro/meshes/simple/hip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 scale=0.001 0.001 0.001; visual mesh filename=package://vir_singlejoint/robots/centauro/meshes/hip-pitch.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 scale=0.001 0.001 0.001
- link hip2_4: geometry collision mesh filename=package://vir_singlejoint/robots/centauro/meshes/simple/hip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 scale=0.001 0.001 0.001; visual mesh filename=package://vir_singlejoint/robots/centauro/meshes/hip-pitch.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 scale=0.001 0.001 0.001
- link knee_1: geometry collision mesh filename=package://vir_singlejoint/robots/centauro/meshes/simple/kne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 scale=0.001 0.001 0.001; visual mesh filename=package://vir_singlejoint/robots/centauro/meshes/knee.stl scale=0.001 0.001 0.001
- link knee_2: geometry collision mesh filename=package://vir_singlejoint/robots/centauro/meshes/simple/kne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 scale=0.001 0.001 0.001; visual mesh filename=package://vir_singlejoint/robots/centauro/meshes/knee.stl scale=0.001 0.001 0.001
- link knee_3: geometry collision mesh filename=package://vir_singlejoint/robots/centauro/meshes/simple/kne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 scale=0.001 0.001 0.001; visual mesh filename=package://vir_singlejoint/robots/centauro/meshes/knee.stl scale=0.001 0.001 0.001
- link knee_4: geometry collision mesh filename=package://vir_singlejoint/robots/centauro/meshes/simple/kne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 scale=0.001 0.001 0.001; visual mesh filename=package://vir_singlejoint/robots/centauro/meshes/knee.stl scale=0.001 0.001 0.001
- link neck_1: geometry collision mesh filename=package://vir_singlejoint/robots/centauro/meshes/simple/nec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 scale=0.001 0.001 0.001; visual mesh filename=package://vir_singlejoint/robots/centauro/meshes/neck_yaw.s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 scale=0.001 0.001 0.001
- link neck_2: geometry collision mesh filename=package://vir_singlejoint/robots/centauro/meshes/simple/nec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 scale=0.001 0.001 0.001; visual mesh filename=package://vir_singlejoint/robots/centauro/meshes/neck_pitch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 scale=0.001 0.001 0.001
- link neck_3: geometry collision mesh filename=package://vir_singlejoint/robots/centauro/meshes/simple/lid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 scale=0.001 0.001 0.001; visual mesh filename=package://vir_singlejoint/robots/centauro/meshes/lidar.stl scale=0.001 0.001 0.001
- link pelvis: geometry collision mesh filename=package://vir_singlejoint/robots/centauro/meshes/simple/pel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 scale=0.001 0.001 0.001; visual mesh filename=package://vir_singlejoint/robots/centauro/meshes/pelvis.stl scale=0.001 0.001 0.001
- link torso_2: geometry collision mesh filename=package://vir_singlejoint/robots/centauro/meshes/simple/lin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 scale=0.001 0.001 0.001; visual mesh filename=package://vir_singlejoint/robots/centauro/meshes/link1.stl scale=0.001 0.001 0.001
- link wheel_1: geometry collision cylinder length=0.06 radius=0.078; visual mesh filename=package://vir_singlejoint/robots/centauro/meshes/wheel.stl scale=0.001 0.001 0.001
- link wheel_2: geometry collision cylinder length=0.06 radius=0.078; visual mesh filename=package://vir_singlejoint/robots/centauro/meshes/wheel.stl scale=0.001 0.001 0.001
- link wheel_3: geometry collision cylinder length=0.06 radius=0.078; visual mesh filename=package://vir_singlejoint/robots/centauro/meshes/wheel.stl scale=0.001 0.001 0.001
- link wheel_4: geometry collision cylinder length=0.06 radius=0.078; visual mesh filename=package://vir_singlejoint/robots/centauro/meshes/wheel.stl scale=0.001 0.001 0.001

Commit message: Revert "added launch file for centauro in cartesio tests quick start"
This reverts commit f81accc2e20e362fedeb6ea35475e14ffda719eb.

File: CartesioTestsQuickStart/robots/centauro/urdf/centauro.urdf (robot description, URDF)
Before this commit: robot centauro, 54 links, 53 joints
Links:
- link ankle1_1: geometry collision mesh filename=package://centauro_urdf/meshes/simple/ankle-pitch.stl scale=0.001 0.001 0.001; visual mesh filename=package://centauro_urdf/meshes/ankle-pitch.stl scale=0.001 0.001 0.001
- link ankle1_2: geometry collision mesh filename=package://centauro_urdf/meshes/simple/ankle-pitch.stl scale=0.001 0.001 0.001; visual mesh filename=package://centauro_urdf/meshes/ankle-pitch.stl scale=0.001 0.001 0.001
- link ankle1_3: geometry collision mesh filename=package://centauro_urdf/meshes/simple/ankle-pitch.stl scale=0.001 0.001 0.001; visual mesh filename=package://centauro_urdf/meshes/ankle-pitch.stl scale=0.001 0.001 0.001
- link ankle1_4: geometry collision mesh filename=package://centauro_urdf/meshes/simple/ankle-pitch.stl scale=0.001 0.001 0.001; visual mesh filename=package://centauro_urdf/meshes/ankle-pitch.stl scale=0.001 0.001 0.001
- link ankle2_1: geometry collision mesh filename=package://centauro_urdf/meshes/simple/ankle-yaw.stl scale=0.001 0.001 0.001; visual mesh filename=package://centauro_urdf/meshes/ankle-yaw.stl scale=0.001 0.001 0.001
- link ankle2_2: geometry collision mesh filename=package://centauro_urdf/meshes/simple/ankle-yaw.stl scale=0.001 0.001 0.001; visual mesh filename=package://centauro_urdf/meshes/ankle-yaw.stl scale=0.001 0.001 0.001
- link ankle2_3: geometry collision mesh filename=package://centauro_urdf/meshes/simple/ankle-yaw.stl scale=0.001 0.001 0.001; visual mesh filename=package://centauro_urdf/meshes/ankle-yaw.stl scale=0.001 0.001 0.001
- link ankle2_4: geometry collision mesh filename=package://centauro_urdf/meshes/simple/ankle-yaw.stl scale=0.001 0.001 0.001; visual mesh filename=package://centauro_urdf/meshes/ankle-yaw.stl scale=0.001 0.001 0.001
- link arm1_1: geometry collision mesh filename=package://centauro_urdf/meshes/simple/ShoulderPitch.STL scale=0.001 -0.001 0.001; visual mesh filename=package://centauro_urdf/meshes/ShoulderPitch.STL scale=0.001 -0.001 0.001
- link arm1_2: geometry collision mesh filename=package://centauro_urdf/meshes/simple/ShoulderRoll.STL scale=0.001 -0.001 0.001; visual mesh filename=package://centauro_urdf/meshes/ShoulderRoll.STL scale=0.001 -0.001 0.001
- link arm1_3: geometry collision mesh filename=package://centauro_urdf/meshes/simple/ShoulderYaw.STL scale=0.001 -0.001 0.001; visual mesh filename=package://centauro_urdf/meshes/ShoulderYaw.STL scale=0.001 -0.001 0.001
- link arm1_4: geometry collision mesh filename=package://centauro_urdf/meshes/simple/Elbow.STL scale=0.001 -0.001 0.001; visual mesh filename=package://centauro_urdf/meshes/Elbow.STL scale=0.001 -0.001 0.001
- link arm1_5: geometry collision mesh filename=package://centauro_urdf/meshes/simple/Forearm.STL scale=0.001 -0.001 0.001; visual mesh filename=package://centauro_urdf/meshes/Forearm.STL scale=0.001 -0.001 0.001
- link arm1_6: geometry collision mesh filename=package://centauro_urdf/meshes/simple/ForearmPitch.STL scale=0.001 -0.001 0.001; visual mesh filename=package://centauro_urdf/meshes/ForearmPitch.STL scale=0.001 -0.001 0.001
- link arm1_7: geometry collision mesh filename=package://centauro_urdf/meshes/simple/ForearmYaw.STL scale=0.001 -0.001 0.001; visual mesh filename=package://centauro_urdf/meshes/ForearmYaw.STL scale=0.001 -0.001 0.001
- link arm2_1: geometry collision mesh filename=package://centauro_urdf/meshes/simple/ShoulderPitch.STL scale=0.001 0.001 0.001; visual mesh filename=package://centauro_urdf/meshes/ShoulderPitch.STL scale=0.001 0.001 0.001
- link arm2_2: geometry collision mesh filename=package://centauro_urdf/meshes/simple/ShoulderRoll.STL scale=0.001 0.001 0.001; visual mesh filename=package://centauro_urdf/meshes/ShoulderRoll.STL scale=0.001 0.001 0.001
- link arm2_3: geometry collision mesh filename=package://centauro_urdf/meshes/simple/ShoulderYaw.STL scale=0.001 0.001 0.001; visual mesh filename=package://centauro_urdf/meshes/ShoulderYaw.STL scale=0.001 0.001 0.001
- link arm2_4: geometry collision mesh filename=package://centauro_urdf/meshes/simple/Elbow.STL scale=0.001 0.001 0.001; visual mesh filename=package://centauro_urdf/meshes/Elbow.STL scale=0.001 0.001 0.001
- link arm2_5: geometry collision mesh filename=package://centauro_urdf/meshes/simple/Forearm.STL scale=0.001 0.001 0.001; visual mesh filename=package://centauro_urdf/meshes/Forearm.STL scale=0.001 0.001 0.001
- link arm2_6: geometry collision mesh filename=package://centauro_urdf/meshes/simple/ForearmPitch.STL scale=0.001 0.001 0.001; visual mesh filename=package://centauro_urdf/meshes/ForearmPitch.STL scale=0.001 0.001 0.001
- link arm2_7: geometry collision mesh filename=package://centauro_urdf/meshes/simple/ForearmYaw.STL scale=0.001 0.001 0.001; visual mesh filename=package://centauro_urdf/meshes/ForearmYaw.STL scale=0.001 0.001 0.001
- link ball1: geometry collision mesh filename=package://centauro_urdf/meshes/simple/BallHand.stl scale=0.001 0.001 0.001; visual mesh filename=package://centauro_urdf/meshes/BallHand.stl scale=0.001 0.001 0.001
- link ball2: geometry collision mesh filename=package://centauro_urdf/meshes/simple/BallHand.stl scale=0.001 0.001 0.001; visual mesh filename=package://centauro_urdf/meshes/BallHand.stl scale=0.001 0.001 0.001
- link hip1_1: geometry collision mesh filename=package://centauro_urdf/meshes/simple/hip-yaw.stl scale=0.001 0.001 0.001; visual mesh filename=package://centauro_urdf/meshes/hip-yaw.stl scale=0.001 0.001 0.001
- link hip1_2: geometry collision mesh filename=package://centauro_urdf/meshes/simple/hip-yaw.stl scale=0.001 0.001 0.001; visual mesh filename=package://centauro_urdf/meshes/hip-yaw.stl scale=0.001 0.001 0.001
- link hip1_3: geometry collision mesh filename=package://centauro_urdf/meshes/simple/hip-yaw.stl scale=0.001 0.001 0.001; visual mesh filename=package://centauro_urdf/meshes/hip-yaw.stl scale=0.001 0.001 0.001
- link hip1_4: geometry collision mesh filename=package://centauro_urdf/meshes/simple/hip-yaw.stl scale=0.001 0.001 0.001; visual mesh filename=package://centauro_urdf/meshes/hip-yaw.stl scale=0.001 0.001 0.001
- link hip2_1: geometry collision mesh filename=package://centauro_urdf/meshes/simple/hip-pitch.stl scale=0.001 0.001 0.001; visual mesh filename=package://centauro_urdf/meshes/hip-pitch.stl scale=0.001 0.001 0.001
- link hip2_2: geometry collision mesh filename=package://centauro_urdf/meshes/simple/hip-pitch.stl scale=0.001 0.001 0.001; visual mesh filename=package://centauro_urdf/meshes/hip-pitch.stl scale=0.001 0.001 0.001
- link hip2_3: geometry collision mesh filename=package://centauro_urdf/meshes/simple/hip-pitch.stl scale=0.001 0.001 0.001; visual mesh filename=package://centauro_urdf/meshes/hip-pitch.stl scale=0.001 0.001 0.001
- link hip2_4: geometry collision mesh filename=package://centauro_urdf/meshes/simple/hip-pitch.stl scale=0.001 0.001 0.001; visual mesh filename=package://centauro_urdf/meshes/hip-pitch.stl scale=0.001 0.001 0.001
- link knee_1: geometry collision mesh filename=package://centauro_urdf/meshes/simple/knee.stl scale=0.001 0.001 0.001; visual mesh filename=package://centauro_urdf/meshes/knee.stl scale=0.001 0.001 0.001
- link knee_2: geometry collision mesh filename=package://centauro_urdf/meshes/simple/knee.stl scale=0.001 0.001 0.001; visual mesh filename=package://centauro_urdf/meshes/knee.stl scale=0.001 0.001 0.001
- link knee_3: geometry collision mesh filename=package://centauro_urdf/meshes/simple/knee.stl scale=0.001 0.001 0.001; visual mesh filename=package://centauro_urdf/meshes/knee.stl scale=0.001 0.001 0.001
- link knee_4: geometry collision mesh filename=package://centauro_urdf/meshes/simple/knee.stl scale=0.001 0.001 0.001; visual mesh filename=package://centauro_urdf/meshes/knee.stl scale=0.001 0.001 0.001
- link neck_1: geometry collision mesh filename=package://centauro_urdf/meshes/simple/neck_yaw.stl scale=0.001 0.001 0.001; visual mesh filename=package://centauro_urdf/meshes/neck_yaw.stl scale=0.001 0.001 0.001
- link neck_2: geometry collision mesh filename=package://centauro_urdf/meshes/simple/neck_pitch.stl scale=0.001 0.001 0.001; visual mesh filename=package://centauro_urdf/meshes/neck_pitch.stl scale=0.001 0.001 0.001
- link neck_3: geometry collision mesh filename=package://centauro_urdf/meshes/simple/lidar.stl scale=0.001 0.001 0.001; visual mesh filename=package://centauro_urdf/meshes/lidar.stl scale=0.001 0.001 0.001
- link pelvis: geometry collision mesh filename=package://centauro_urdf/meshes/simple/pelvis.stl scale=0.001 0.001 0.001; visual mesh filename=package://centauro_urdf/meshes/pelvis.stl scale=0.001 0.001 0.001
- link torso_2: geometry collision mesh filename=package://centauro_urdf/meshes/simple/link1.stl scale=0.001 0.001 0.001; visual mesh filename=package://centauro_urdf/meshes/link1.stl scale=0.001 0.001 0.001
- link wheel_1: geometry collision cylinder length=0.06 radius=0.078; visual mesh filename=package://centauro_urdf/meshes/wheel.stl scale=0.001 0.001 0.001
- link wheel_2: geometry collision cylinder length=0.06 radius=0.078; visual mesh filename=package://centauro_urdf/meshes/wheel.stl scale=0.001 0.001 0.001
- link wheel_3: geometry collision cylinder length=0.06 radius=0.078; visual mesh filename=package://centauro_urdf/meshes/wheel.stl scale=0.001 0.001 0.001
- link wheel_4: geometry collision cylinder length=0.06 radius=0.078; visual mesh filename=package://centauro_urdf/meshes/wheel.stl scale=0.001 0.001 0.001
